Commit message: First trial

File: urdf/turtlebot3_burger.urdf (robot description, URDF)
Before this commit: robot turtlebot3_burger, 7 links, 6 joints
Links:
- added link camera_link, mass 0.035; collision box size=0.015 0.030 0.027; visual box size=0.015 0.030 0.027
Joints:
- added joint camera_joint: type continuous, parent base_link, child camera_link, origin xyz=-0.032 0 0.192 rpy=0 0 0
