Commit message: Update camera joint position in URDF and enhance camera field of view calculations in simulation node. Adjust vertical and horizontal FOV for improved rendering accuracy and add debug print for camera settings.

File: data/urdf/turtlebot3_burger.urdf (robot description, URDF)
Before this commit: robot turtlebot3_burger, 8 links, 7 joints
Joints:
- joint camera_joint: origin xyz=-0.032 0 0.192 rpy=0 0 0 -> xyz=0.05 0 0.192 rpy=0 0 0
