Commit message: Structure urdf properly for starting the sim

File: data/urdf/maurice.urdf (robot description, URDF)
Before this commit: robot maurice_bot, 13 links, 12 joints
Links:
- link arm_camera_link: geometry visual sphere radius=0.005
- link base_link: geometry collision box size=0.1878 0.182 0.1676; visual mesh filename=meshes/base.STL scale=1 1 1
- link link1: geometry collision mesh filename=meshes/link1.STL scale=1 1 1; visual mesh filename=meshes/link1.STL scale=1 1 1
- link link2: geometry collision box size=0.020 0.054 0.1385; visual mesh filename=meshes/link2.STL scale=1 1 1
- link link3: geometry collision cylinder length=0.118 radius=0.023; visual mesh filename=meshes/link3.STL scale=1 1 1
- link link4: geometry collision mesh filename=meshes/link4.STL scale=1 1 1; visual mesh filename=meshes/link4.STL scale=1 1 1
- link link5: geometry collision mesh filename=meshes/link5.STL scale=0.001 0.001 0.001; visual mesh filename=meshes/link5.STL scale=0.001 0.001 0.001
- link link61: geometry collision box size=0.048 0.016 0.0389; visual mesh filename=meshes/link61.STL scale=0.001 0.001 0.001
- link link62: geometry collision box size=0.048 0.016 0.0389; visual mesh filename=meshes/link62.STL scale=0.001 0.001 0.001
Joints:
- removed joint fixed_arm_camera_link
- added joint arm_camera_joint: type revolute, parent link5, child arm_camera_link, origin xyz=0.00454 0 0.05448 rpy=0 0 0, axis 0 0 1, limit lower=0 upper=0 effort=0 velocity=0

Commit message: Add head camera link to URDF and implement arm joint position control via ROS bridge

File: data/urdf/maurice.urdf (robot description, URDF)
Before this commit: robot maurice_bot, 13 links, 12 joints
Links:
- added link head_camera_link, mass 0.01; visual sphere radius=0.01
Joints:
- added joint head_camera_joint: type revolute, parent base_link, child head_camera_link, origin xyz=0 0 0.20 rpy=0 0 0, axis 0 0 1, limit lower=0 upper=0 effort=0 velocity=0
