Commit message: camera link

File: ros2_ws/src/maurice_bot/maurice_sim/urdf/maurice.urdf (robot description, URDF)
Before this commit: robot maurice_bot, 8 links, 7 joints
Links:
- added link arm_camera_link, mass 0.01
Joints:
- added joint arm_camera_joint: type fixed, parent link5, child arm_camera_link, origin xyz=0.00454 0 0.05448 rpy=0 0.802851 0

Commit message: using pure pykdly now

File: ros2_ws/src/maurice_bot/maurice_sim/urdf/maurice.urdf (robot description, URDF)
Before this commit: robot maurice_bot, 11 links, 10 joints
Links:
- link base_root: mass 0.01 -> None

Commit message: new ee link

File: ros2_ws/src/maurice_bot/maurice_sim/urdf/maurice.urdf (robot description, URDF)
Before this commit: robot maurice_bot, 11 links, 10 joints
Links:
- added link ee_link, mass 0.001; visual sphere radius=0.005
Joints:
- added joint ee_joint: type fixed, parent link5, child ee_link, origin xyz=0.065 0 0 rpy=0 0 0

Commit message: link 1 collision correct

File: ros2_ws/src/maurice_bot/maurice_sim/urdf/maurice.urdf (robot description, URDF)
Before this commit: robot maurice_bot, 13 links, 12 joints
Links:
- link base_link: geometry collision box size=0.1878 0.182 0.1676; visual mesh filename=package://maurice_sim/meshes/base.STL scale=1 1 1

Commit message: Updated URDF, meshes outdated
Having some trouble exporting proper meshes even with everything properly selected in the exporter.

File: ros2_ws/src/maurice_bot/maurice_sim/urdf/maurice.urdf (robot description, URDF)
Before this commit: robot maurice_bot, 13 links, 12 joints
Links:
- added link head, mass 0.148; collision mesh filename=package://maurice_sim/meshes/head.STL scale=1 1 1; visual mesh filename=package://maurice_sim/meshes/head.STL scale=1 1 1
- added link head_camera_left, mass 0.01; visual sphere radius=0.005
- added link head_camera_right, mass 0.01; visual sphere radius=0.005
Joints:
- added joint fixed_head_camera_left: type fixed, parent head, child head_camera_left, origin xyz=0.04327 0.0297 -0.000275 rpy=0 0 0
- added joint fixed_head_camera_right: type fixed, parent head, child head_camera_right, origin xyz=0.04327 -0.0303 -0.000275 rpy=0 0 0
- added joint joint_head: type fixed, parent base_link, child head, origin xyz=-0.040751 -0.0002 0.25882 rpy=0 0 0
- joint ee_joint: origin xyz=0.09285 0 0 rpy=0 0 0 -> xyz=0.0887 0 0 rpy=0 0 0
- joint fixed_arm_camera_link: origin xyz=0.00454 0 0.05448 rpy=0 0 0 -> xyz=0.03378 0 0.05052 rpy=0 0.43633 0
- joint joint2: origin xyz=0 0 0.04225 rpy=0 0 0 -> xyz=0 0 0.04425 rpy=0 0 0
- joint joint4: origin xyz=0.1375 0 -0.0045 rpy=0 0 0 -> xyz=0.1375 0 0.0045 rpy=0 0 0
- joint joint6: origin xyz=0.044 -0.0091 0 rpy=0 0 0 -> xyz=0.044 -0.0092 0 rpy=0 0 0

Commit message: Unify TF publishing through robot_state_publisher
- URDF: Rename base_root to odom for proper TF chain
- i2c.py: Store odom_x, odom_y, odom_yaw directly (simplified)
- i2c.py: Remove TransformStamped, use simple float values
- bringup.py: Publish base_x, base_y, base_yaw to /joint_states
- bringup.py: Remove direct TF broadcast, let robot_state_publisher handle it
- bringup.py: Keep /odom topic for Nav2 velocity info

File: ros2_ws/src/maurice_bot/maurice_sim/urdf/maurice.urdf (robot description, URDF)
Before this commit: robot maurice_bot, 16 links, 15 joints
Links:
- removed link base_root
- added link odom
Joints:
- joint base_x: parent base_root -> odom

Commit message: Revert i2c.py and bringup.py to main, maurice.urdf to URDF_Update

File: ros2_ws/src/maurice_bot/maurice_sim/urdf/maurice.urdf (robot description, URDF)
Before this commit: robot maurice_bot, 16 links, 15 joints
Links:
- removed link odom
- added link base_root
Joints:
- joint base_x: parent odom -> base_root

Commit message: URDF Rotation fixed, head rotation config reverted

File: ros2_ws/src/maurice_bot/maurice_sim/urdf/maurice.urdf (robot description, URDF)
Before this commit: robot maurice_bot, 13 links, 12 joints
Joints:
- joint joint6: axis 0 0 1 -> 0 0 -1
- joint joint6M: axis 0 0 1 -> 0 0 -1
- joint joint_head: axis 0 1 0 -> 0 -1 0

Commit message: updating ee_link to be at the tip of link6 instead of middle of flat section

File: ros2_ws/src/maurice_bot/maurice_sim/urdf/maurice.urdf (robot description, URDF)
Before this commit: robot maurice_bot, 13 links, 12 joints
Joints:
- joint ee_joint: origin xyz=0.0887 0 0 rpy=0 0 0 -> xyz=0.091838 0 0 rpy=0 0 0

Commit message: adding collision boxes to URDF

File: ros2_ws/src/maurice_bot/maurice_sim/urdf/maurice.urdf (robot description, URDF)
Before this commit: robot maurice_bot, 13 links, 12 joints
Links:
- link head: geometry collision box size=0.113 0.121 0.036; visual mesh filename=package://maurice_sim/meshes/head.STL scale=1 1 1
- link link1: geometry collision box size=0.067 0.040 0.082; visual mesh filename=package://maurice_sim/meshes/link1.STL scale=1 1 1
- link link2: geometry collision box size=0.037 0.054 0.156; visual mesh filename=package://maurice_sim/meshes/link2.STL scale=1 1 1
- link link3: geometry collision box size=0.134 0.054 0.035; visual mesh filename=package://maurice_sim/meshes/link3.STL scale=1 1 1
- link link4: geometry collision box size=0.032 0.039 0.020; visual mesh filename=package://maurice_sim/meshes/link4.STL scale=1 1 1
- link link5: geometry collision box size=0.054 0.044 0.093; visual mesh filename=package://maurice_sim/meshes/link5.STL scale=1 1 1

Commit message: transform

File: ros2_ws/src/maurice_bot/maurice_sim/urdf/maurice.urdf (robot description, URDF)
Before this commit: robot maurice_bot, 13 links, 12 joints
Links:
- added link camera_optical_frame
Joints:
- added joint fixed_camera_optical_frame: type fixed, parent head_camera_left, child camera_optical_frame, origin xyz=0 0 0 rpy=-1.5708 0 -1.5708

Commit message: make stereo work through ros pipeline as well

File: ros2_ws/src/maurice_bot/maurice_sim/urdf/maurice.urdf (robot description, URDF)
Before this commit: robot maurice_bot, 14 links, 13 joints
Links:
- added link right_camera_optical_frame
Joints:
- added joint fixed_right_camera_optical_frame: type fixed, parent head_camera_right, child right_camera_optical_frame, origin xyz=0 0 0 rpy=-1.5708 0 -1.5708

Commit message: Update URDF with proper inertia and mass, add wheels, separate actuators from links
- Add accurate mass and inertia tensors from SolidWorks for all plastic links
- Separate Dynamixel motors (m2-m6) into dedicated links with fixed joints
- Add left/right wheel links with continuous joints rotating around Y axis
- Add caster wheel assembly (frame + wheel) with proper swivel mechanics
- Update head link with correct physical properties
- Include new mesh files for wheels, caster, and motor housings

Made-with: Cursor

File: ros2_ws/src/maurice_bot/maurice_sim/urdf/maurice.urdf (robot description, URDF)
Before this commit: robot maurice_bot, 15 links, 14 joints
Links:
- added link caster_frame, mass 0.0147; collision mesh filename=package://maurice_sim/meshes/caster_frame.STL scale=1 1 1; visual mesh filename=package://maurice_sim/meshes/caster_frame.STL scale=1 1 1
- added link caster_wheel, mass 0.0106; collision sphere radius=0.01235; visual mesh filename=package://maurice_sim/meshes/caster_wheel.STL scale=1 1 1
- added link left_wheel, mass 0.26; collision cylinder length=0.02 radius=0.03725; visual mesh filename=package://maurice_sim/meshes/left_wheel.STL scale=1 1 1
- added link m2, mass 0.065; collision mesh filename=package://maurice_sim/meshes/m2.STL scale=1 1 1; visual mesh filename=package://maurice_sim/meshes/m2.STL scale=1 1 1
- added link m3, mass 0.057; collision mesh filename=package://maurice_sim/meshes/m3.STL scale=1 1 1; visual mesh filename=package://maurice_sim/meshes/m3.STL scale=1 1 1
- added link m4, mass 0.023; collision mesh filename=package://maurice_sim/meshes/m4.STL scale=1 1 1; visual mesh filename=package://maurice_sim/meshes/m4.STL scale=1 1 1
- added link m5, mass 0.023; collision mesh filename=package://maurice_sim/meshes/m5.STL scale=1 1 1; visual mesh filename=package://maurice_sim/meshes/m5.STL scale=1 1 1
- added link m6, mass 0.023; collision mesh filename=package://maurice_sim/meshes/m6.STL scale=1 1 1; visual mesh filename=package://maurice_sim/meshes/m6.STL scale=1 1 1
- added link right_wheel, mass 0.26; collision cylinder length=0.02 radius=0.03725; visual mesh filename=package://maurice_sim/meshes/right_wheel.STL scale=1 1 1
- link arm_camera_link: mass 0.01 -> 0.00649
- link base_link: mass 0.89 -> 1.435
- link head: mass 0.148 -> 0.1338
- link link1: mass 0.065 -> 0.0288
- link link2: mass 0.080 -> 0.039
- link link3: mass 0.055 -> 0.0366
- link link4: mass 0.022 -> 0.00841
- link link5: mass 0.050 -> 0.0383
- link link61: mass 0.012 -> 0.00731
- link link62: mass 0.012 -> 0.00730
Joints:
- added joint caster_frame_joint: type continuous, parent base_link, child caster_frame, origin xyz=-0.1229 0 0.037775 rpy=0 0 0, axis 0 0 1
- added joint caster_wheel_joint: type continuous, parent caster_frame, child caster_wheel, origin xyz=-0.0085 0 -0.025425 rpy=0 0 0, axis 0 1 0
- added joint left_wheel_joint: type continuous, parent base_link, child left_wheel, origin xyz=0 0.0882 0.03725 rpy=0 0 0, axis 0 1 0
- added joint m2_joint: type fixed, parent link1, child m2, origin xyz=0 -0.019 0.04425 rpy=1.5708 1.5708 0
- added joint m3_joint: type fixed, parent link2, child m3, origin xyz=0.02825 -0.019 0.12125 rpy=1.5708 1.5708 0
- added joint m4_joint: type fixed, parent link3, child m4, origin xyz=0.1375 -0.0145 0.0045 rpy=1.5708 1.5708 0
- added joint m5_joint: type fixed, parent link5, child m5, origin xyz=0 0 0 rpy=-1.5708 0 1.5708
- added joint m6_joint: type fixed, parent link5, child m6, origin xyz=0.044 0.0091 -0.0145 rpy=3.1416 0 -3.1416
- added joint right_wheel_joint: type continuous, parent base_link, child right_wheel, origin xyz=0 -0.0882 0.03725 rpy=0 0 0, axis 0 1 0
- joint joint6: limit lower=-0.8727 upper=0.3491 effort=2.0 velocity=2.0 -> lower=0 upper=0.9076 effort=2.0 velocity=2.0
- joint joint6M: limit lower=-0.8727 upper=0.3491 effort=2.0 velocity=2.0 -> lower=-0.9076 upper=0 effort=2.0 velocity=2.0

Commit message: Add effort/velocity limits to wheel and caster joints
- Hub motor joints: effort=0.25 N·m (rated), velocity=10.3 rad/s (98 rpm)
- Caster joints: passive (effort=0), velocity=100 rad/s, friction=0.1
- Required by diff_drive_controller and Gazebo plugins

Made-with: Cursor

File: ros2_ws/src/maurice_bot/maurice_sim/urdf/maurice.urdf (robot description, URDF)
Before this commit: robot maurice_bot, 24 links, 23 joints
Joints:
- joint caster_frame_joint: limit (none) -> effort=0.0 velocity=100.0
- joint caster_wheel_joint: limit (none) -> effort=0.0 velocity=100.0
- joint left_wheel_joint: limit (none) -> effort=0.25 velocity=10.3
- joint right_wheel_joint: limit (none) -> effort=0.25 velocity=10.3

Commit message: zeno-ram-usage

File: ros2_ws/src/maurice_bot/maurice_sim/urdf/maurice.urdf (robot description, URDF)
Before this commit: robot maurice_bot, 15 links, 14 joints
Links:
- added link base_footprint
- added link base_laser
Joints:
- added joint base_footprint_joint: type fixed, parent base_link, child base_footprint, origin xyz=0 0 0 rpy=0 0 0
- added joint base_laser_joint: type fixed, parent base_link, child base_laser, origin xyz=-0.0764 0.0 0.17165 rpy=0 0 0

Commit message: hello

File: ros2_ws/src/maurice_bot/maurice_sim/urdf/maurice.urdf (robot description, URDF)
Before this commit: robot maurice_bot, 17 links, 16 joints
Links:
- removed link base_footprint
- removed link base_laser
Joints:
- removed joint base_footprint_joint
- removed joint base_laser_joint
