Commit message: increase upward tilt to 35 degrees

File: ros2_ws/src/mars_bot/mars_sim/urdf/mars.urdf (robot description, URDF)
Before this commit: robot mars_bot, 17 links, 16 joints
Joints:
- joint joint_head: limit lower=-0.3491 upper=0.3491 effort=2.0 velocity=2.0 -> lower=-0.3491 upper=0.6109 effort=2.0 velocity=2.0
