Commit message: refactor: rename mars_sim to mars_description
mars_sim contains no simulation. It is the robot description -- mars.urdf,
arm.srdf and nine STL meshes -- and mars_arm, mars_bringup and mars_sim_driver
all exec_depend on it, so it is load-bearing on real hardware, not just in sim.
Its own package.xml already said as much.

The name was the single biggest source of the "three simulators" confusion: a
newcomer reads mars_sim as the simulator and mars_sim_driver as its driver, when
it is the other way round. mars_description is the ROS convention.

44 occurrences across 21 files, all verified as the package name rather than the
mars_sim_driver / mars_sim_bringup prefixes. Four of them have to agree with one
another and now do: the package:// URIs in mars.urdf, scene.ts's
`loader.packages` key, viz.js's replace target, and the proxy's /robot/ route.

Note: sim/launcher/config.py names the package path in both the assets-image
input list and NON_GEOMETRY_PATHSPECS, so this renames the asset image; `up`
falls back to a local build until CI publishes the new hash.

File: ros2_ws/src/mars_bot/mars_description/urdf/mars.urdf (robot description, URDF)
Before this commit: robot mars_bot, 17 links, 16 joints
Links:
- link base_link: geometry collision box size=0.0374 0.036 0.0366; collision box size=0.051 0.0854 0.039
- link head: geometry collision box size=0.113 0.121 0.036; visual mesh filename=package://mars_description/meshes/head.STL scale=1 1 1
- link link1: geometry collision box size=0.0403 0.0226 0.0466; collision box size=0.0465 0.04 0.0216
- link link2: geometry collision box size=0.0244 0.0475 0.0436; collision box size=0.035 0.054 0.0763
- link link3: geometry collision box size=0.028 0.0467 0.031; collision box size=0.0677 0.054 0.035
- link link4: geometry collision box size=0.032 0.039 0.020; visual mesh filename=package://mars_description/meshes/link4.STL scale=1 1 1
- link link5: geometry collision box size=0.054 0.044 0.093; visual mesh filename=package://mars_description/meshes/link5.STL scale=1 1 1
- link link61: geometry collision box size=0.0022 0.0045 0.0389; collision box size=0.0022 0.0062 0.0389
- link link62: geometry collision box size=0.0022 0.0045 0.0389; collision box size=0.0022 0.0062 0.0389

Commit message: fix(arm): joint2-4 limits in the URDF are the servo's, negated like joint6
arm_control.cpp negates joints 2, 3, 4 and 6 between the servo and ROS, and
the servo enforces arm_config.yaml's raw position_limits. The URDF converted
joint6's range (see its note) but copied 2-4 verbatim, so every range was
mirrored: the IK (since #740, which rejects out-of-limit solutions) refused
poses the arm reaches and accepted ones the servo clamps. The rest pose sits
exactly on the corrected stops (joint2 -1.2195 vs -1.22, joint3 1.5723 vs
1.5708).

Replayed through the KDL solver with main's ik.py seeding and check:
- drop_in_box's release band (x 0.24-0.34, y +-0.10, z 0.10-0.27, pitch 1.30):
  597 -> 818 of 990 solved, none clamped by the servo. The failing robot drop
  at (0.32, -0.04, 0.15) now solves with joint4 = 1.922.
- The #740 hazard, a small lift from rest: accepted and mis-executed before
  (+3 cm asked, +1.4 cm landed), refused now.

The Arm SDK page's sliders carried a copy of the mirrored ranges; corrected
too. The sim loads this URDF as the arm's hard stops, so its start pose is
checked separately.

File: ros2_ws/src/mars_bot/mars_description/urdf/mars.urdf (robot description, URDF)
Before this commit: robot mars_bot, 17 links, 16 joints
Joints:
- joint joint2: limit lower=-1.5708 upper=1.22 effort=2.0 velocity=2.0 -> lower=-1.22 upper=1.5708 effort=2.0 velocity=2.0
- joint joint3: limit lower=-1.5708 upper=1.7453 effort=2.0 velocity=2.0 -> lower=-1.7453 upper=1.5708 effort=2.0 velocity=2.0
- joint joint4: limit lower=-1.9199 upper=1.7453 effort=2.0 velocity=2.0 -> lower=-1.7453 upper=1.9199 effort=2.0 velocity=2.0
